Commit message: New class for robot UR10e has been added, taking the same structure as UR5e. URDF file has been slightly modified and collision and visuals meshes have been added. New class tested and working. 31-03

File: rm4d/robots/assets/ur10e.urdf (robot description, URDF)
Before this commit: robot ur10e, 13 links, 12 joints
Links:
- link base_link_inertia: geometry collision mesh filename=meshes/ur10e/collision/base.stl; visual mesh filename=meshes/ur10e/visual/base.dae
- link forearm_link: geometry collision mesh filename=meshes/ur10e/collision/forearm.stl; visual mesh filename=meshes/ur10e/visual/forearm.dae
- link shoulder_link: geometry collision mesh filename=meshes/ur10e/collision/shoulder.stl; visual mesh filename=meshes/ur10e/visual/shoulder.dae
- link upper_arm_link: geometry collision mesh filename=meshes/ur10e/collision/upperarm.stl; visual mesh filename=meshes/ur10e/visual/upperarm.dae
- link wrist_1_link: geometry collision mesh filename=meshes/ur10e/collision/wrist1.stl; visual mesh filename=meshes/ur10e/visual/wrist1.dae
- link wrist_2_link: geometry collision mesh filename=meshes/ur10e/collision/wrist2.stl; visual mesh filename=meshes/ur10e/visual/wrist2.dae
- link wrist_3_link: geometry collision mesh filename=meshes/ur10e/collision/wrist3.stl; visual mesh filename=meshes/ur10e/visual/wrist3.dae
